File: RoboBallersLinePCB.kicad_sch (KiCad schematic)
At the start: 116 parts, among them J1 Conn_01x04, J2 Bottom PCB, Q1 P-Channel, Q2 N-Channel, U1 MCP3008, U2 MCP3008, U3 MCP3008, U4 BoostConverter, U5 NSL-32, U6 NSL-32

Commit message: Idk if the changes didnt save
Correct version is this one or something else
Parts:
- added U7: Solenoid-Electric, KickerPad:KickerPad, symbol Solenoid:Solenoid-Electric
Connections:
- net at D49.1 (A), Q2.2 (D): now also U7.2 (GND)
- net at C1.1, D49.2 (K), Q1.2 (D): now also U7.1 (VCC)
Changed lines of the file:
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@@
+	)
+	(symbol
+		(lib_id "Solenoid:Solenoid-Electric")
+		(at 306.07 81.28 0)
+		(unit 1)
+		(exclude_from_sim no)
+		(in_bom yes)
+		(on_board yes)
+		(dnp no)
+		(property "Reference" "U7"
+			(at 299.72 73.66 0)
+			(effects
+				(font
+					(size 1.27 1.27)
+				)
+				(justify left)
+			)
+		)
+		(property "Value" "Solenoid-Electric"
+			(at 290.83 69.85 0)
+			(effects
+				(font
+					(size 1.27 1.27)
+				)
+				(justify left)
+			)
+		)
+		(property "Footprint" "KickerPad:KickerPad"
+			(at 303.53 83.82 0)
+			(effects
+				(font
+					(size 1.27 1.27)
+				)
+				(hide yes)
+			)
+		)
+		(property "Datasheet" ""
+			(at 303.53 83.82 0)
+			(effects
+				(font
+					(size 1.27 1.27)
+				)
+				(hide yes)
+			)
+		)
+		(property "Description" ""
+			(at 306.07 81.28 0)
+			(effects
+				(font
+					(size 1.27 1.27)
+				)
+				(hide yes)
+			)
+		)
+		(pin "1"
+		)
+		(pin "2"
+		)
+		(instances
+			(project "RoboBallersLinePCB"
+				(path "/e29be779-79a0-4fa4-991c-37a1a544ca10"
+					(reference "U7")
+					(unit 1)
+				)
+			)
+		)
 	)
 	(symbol
