File: _autosave-RoboBallersLinePCB.kicad_pcb (KiCad board)
At the start: 2 copper layers, 132 x 132 mm, 117 parts, among them J1 Conn_01x04, J2 Bottom PCB, Q1 P-Channel, Q2 N-Channel, U1 MCP3008, U2 MCP3008, U3 MCP3008, U4 BoostConverter, U5 NSL-32, U6 NSL-32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

Commit message: stoopid 0.2mm -> 1 mm
 - Fixed 90 errors, now realized need to change traces from 0.2mm to 1 mm
Routing:
- net CH43: track 78.8 -> 130.1 mm, vias 0 -> 2
- net CH63: track 40.9 -> 35.8 mm
- net CH23: track 102.8 -> 101.8 mm
