File: RoboBallersLinePCB.kicad_pcb (KiCad board)
At the start: 2 copper layers, 132 x 132 mm, 117 parts, among them J1 Conn_01x04, J2 Bottom PCB, Q1 P-Channel, Q2 N-Channel, U1 MCP3008, U2 MCP3008, U3 MCP3008, U4 BoostConverter, U5 NSL-32, U6 NSL-32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

Commit message: I am better than Spem
- He coulndt do 3.3v

HAAHAHAHAHHA

I AM BETTER
Routing:
- net 3.3v: track 449.7 -> 566.3 mm, vias 4 -> 9
- net GND: track 662.0 -> 713.9 mm, vias 5 -> 7
- net CH43: track 78.8 -> 130.1 mm, vias 0 -> 2
- net CH42: track 26.2 -> 30.2 mm
- net CH63: track 40.9 -> 44.1 mm
- net CH12: track 52.2 -> 54.4 mm
- net CH11: track 50.4 -> 51.3 mm
- net CH53: track 66.9 -> 66.2 mm

Commit message: spem needs to try
Routing:
- added copper zone on B.Cu, net GND
- added copper zone on F.Cu, net GND
Changed lines of the file:
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@@
 		(tags "Through hole vertical IDC box header THT 2x05 2.54mm double row")
 		(property "Reference" "J2"
-			(at 1.27 -6.1 360)
+			(at 1.27 -6.1 0)
 			(layer "F.SilkS")
 			(effects
@@
 		)
 		(property "Value" "Bottom PCB"
-			(at 1.27 16.26 360)
+			(at 1.27 16.26 0)
 			(layer "F.Fab")
 			(effects
@@
 		(net 68)
 	)
+	(zone
+		(net 2)
+		(net_name "GND")
+		(layers "F&B.Cu")
+		(hatch edge 0.5)
+		(connect_pads
+			(clearance 0.5)
+		)
+		(min_thickness 0.25)
+		(filled_areas_thickness no)
+		(fill yes
+			(thermal_gap 0.5)
+			(thermal_bridge_width 0.5)
+		)
+		(polygon
+			(pts
+				(xy 202.6412 214.122) (xy 372.872 210.4136) (xy 382.3716 386.3848) (xy 192.1256 393.192)
+			)
+		)
+	)
 	(group ""

Commit message: prem really did not cook so i had to cook
Routing:
- net Net-(D49-K): track 110.3 -> 138.2 mm, vias 3 -> 15
- net 3.3v: track 566.3 -> 562.0 mm
- net Net-(D49-A): track 52.3 -> 54.9 mm, vias 2 -> 6
- net CH63: track 44.1 -> 42.1 mm
- net Net-(Q2-G): track 97.3 -> 96.2 mm, vias 1 -> 3
- net CH03: track 177.6 -> 176.7 mm

Commit message: nicve
Parts:
- removed J1: Conn_01x04, Connector_PinHeader_2.54mm:PinHeader_1x04_P2.54mm_Vertical
- R7: value 165 -> 750
Routing:
- net GND: track 713.9 -> 687.4 mm
- net 12v: track 145.5 -> 121.1 mm
- net 3.3v: track 562.0 -> 546.0 mm
- net Kicker: track 105.9 -> 93.5 mm

Commit message: redid whole pcb
Parts:
- R52: moved to B.Cu
- moved D48 129.8 mm to (226.9, 310.1), turned to -172 degrees
- moved R26 129.8 mm to (227.5, 313.8), turned to -169 degrees
- moved R51 129.8 mm to (226.5, 306.5), turned to -176 degrees
- moved D24 129.8 mm to (228.3, 317.3), turned to -165 degrees
- moved D1 129.7 mm to (226.4, 302.8), turned to 180 degrees
- moved R50 129.6 mm to (229.4, 320.8), turned to -161 degrees
- moved R2 129.5 mm to (226.5, 299.2), turned to 176 degrees
- moved D47 129.4 mm to (230.6, 324.3), turned to -157 degrees
- moved D25 129.2 mm to (226.9, 295.5), turned to 173 degrees
- moved R25 129.2 mm to (232.2, 327.6), turned to -154 degrees
- moved R28 128.9 mm to (227.5, 291.9), turned to 169 degrees
- moved D23 128.8 mm to (233.9, 330.8), turned to -150 degrees
- moved D2 128.5 mm to (228.3, 288.3), turned to 165 degrees
- moved R49 128.4 mm to (235.8, 333.9), turned to -146 degrees
- moved R3 128.0 mm to (229.4, 284.8), turned to 161 degrees
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Routing:
- net 48v: track 65.7 -> 278.3 mm, vias 0 -> 8
- net CH71: track 63.7 -> 276.0 mm, vias 2 -> 0
- net Net-(Q1-G): track 39.2 -> 230.9 mm, vias 1 -> 18
- net Net-(Q2-G): track 96.2 -> 251.4 mm, vias 3 -> 35
- net Net-(U6-A): track 12.3 -> 141.5 mm, vias 0 -> 2
- net CSLS2: track 55.8 -> 180.9 mm, vias 0 -> 4
- net Net-(U5-A): track 15.6 -> 110.5 mm, vias 0 -> 2
- net GND: track 687.4 -> 609.7 mm, vias 7 -> 23
- net CH03: track 176.7 -> 101.7 mm, vias 4 -> 2
- net CH43: track 130.1 -> 66.7 mm, vias 2 -> 0
- net Net-(D49-K): track 138.2 -> 195.4 mm, vias 15 -> 8
- net 12v: track 121.1 -> 67.2 mm
- net CH22: track 25.0 -> 76.8 mm
- net CH32: track 16.2 -> 65.0 mm
- net CH72: track 67.5 -> 25.8 mm, vias 0 -> 1
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Other:
- outline, holes or cut-outs redrawn

Commit message: !
Parts:
- moved Q2 1.40 mm to (327.3, 326.6)
Routing:
- net GND: track 609.7 -> 675.7 mm
- net Net-(D49-A): track 84.8 -> 83.2 mm
Changed lines of the file:
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@@
 	(footprint "Package_TO_SOT_THT:TO-220-3_Vertical"
 		(layer "F.Cu")
-		(at 327.3044 325.2418 180)
+		(at 327.3044 326.644 180)
 		(descr "TO-220-3, Vertical, RM 2.54mm, see https://www.vishay.com/docs/66542/to-220-1.pdf")
 		(tags "TO-220-3 Vertical RM 2.54mm")
@@
 	)
 	(segment
-		(start 322.2244 324.1368)
-		(end 322.2244 325.2418)
-		(width 0.2)
-		(layer "F.Cu")
-		(net 2)
-	)
-	(segment
 		(start 339.2932 292.4556)
 		(end 335.4324 288.5948)
@@
 	)
 	(segment
-		(start 316.0978 325.2418)
-		(end 322.2244 325.2418)
-		(width 0.2)
-		(layer "F.Cu")
-		(net 2)
-	)
-	(segment
 		(start 336.3976 281.7368)
 		(end 336.3976 284.48)
@@
 	)
 	(segment
-		(start 312.5216 321.6656)
-		(end 316.0978 325.2418)
+		(start 322.2244 324.1368)
+		(end 322.2244 326.644)
 		(width 0.2)
 		(layer "F.Cu")
@@
 	)
 	(segment
+		(start 316.0978 325.2418)
+		(end 320.8222 325.2418)
+		(width 0.2)
+		(layer "F.Cu")
+		(net 2)
+	)
+	(segment
 		(start 259.521165 272.4912)
 		(end 261.3152 272.4912)
@@
 	)
 	(segment
+		(start 320.8222 325.2418)
+		(end 322.2244 326.644)
+		(width 0.2)
+		(layer "F.Cu")
+		(net 2)
+	)
+	(segment
 		(start 259.6488 278.1708)
 		(end 258.1988 276.7208)
@@
 	)
 	(segment
+		(start 312.5216 321.6656)
+		(end 316.0978 325.2418)
+		(width 0.2)
+		(layer "F.Cu")
+		(net 2)
+	)
+	(segment
 		(start 271.9832 245.9228)
 		(end 268.1732 249.7328)
@@
 	)
 	(segment
+		(start 288.323646 355.44516)
+		(end 296.125283 355.44516)
+		(width 0.2)
+		(layer "B.Cu")
+		(net 2)
+	)
+	(segment
 		(start 271.6784 265.5824)
 		(end 271.6784 268.1224)
@@
 	)
 	(segment
+		(start 271.7746 306.7852)
+		(end 271.7746 338.896114)
+		(width 0.2)
+		(layer "B.Cu")
+		(net 2)
+	)
+	(segment
 		(start 271.76383 358.270343)
 		(end 276.595378 358.270343)
@@
 	)
 	(segment
+		(start 271.7746 338.896114)
+		(end 288.323646 355.44516)
+		(width 0.2)
+		(layer "B.Cu")
+		(net 2)
+	)
+	(segment
 		(start 241.118557 265.231138)
 		(end 238.569901 267.779794)
@@
 	)
 	(segment
+		(start 296.125283 355.44516)
+		(end 296.604975 355.924852)
+		(width 0.2)
+		(layer "B.Cu")
+		(net 2)
+	)
+	(segment
 		(start 254.89835 255.236301)
 		(end 255.32843 255.666381)
@@
 	)
 	(segment
+		(start 324.7769 327.7491)
+		(end 324.7769 326.6565)
+		(width 2.75)
+		(layer "F.Cu")
+		(net 28)
+	)
+	(segment
+		(start 324.7769 326.6565)
+		(end 324.7644 326.644)
+		(width 2.75)
+		(layer "F.Cu")
+		(net 28)
+	)
+	(segment
 		(start 323.1388 329.3872)
 		(end 324.7769 327.7491)
@@
 	)
 	(segment
-		(start 324.7769 327.7491)
-		(end 324.7769 325.0184)
-		(width 2.75)
-		(layer "F.Cu")
-		(net 28)
-	)
-	(segment
 		(start 301.7546 328.749042)
 		(end 301.7546 333.0372)
@@
 	)
 	(segment
+		(start 327.3044 326.644)
+		(end 327.3044 297.9928)
+		(width 2.5)
+		(layer "B.Cu")
+		(net 34)
+	)
+	(segment
 		(start 284.3784 260.9596)
 		(end 283.972 261.366)
@@
 	)
 	(segment
-		(start 327.3044 297.9928)
-		(end 322.072 292.7604)
-		(width 2.5)
+		(start 277.114 312.8264)
+		(end 277.114 311.3024)
+		(width 2.75)
 		(layer "B.Cu")
 		(net 34)
 	)
 	(segment
-		(start 277.114 312.8264)
-		(end 277.114 311.3024)
-		(width 2.75)
+		(start 327.3044 297.9928)
+		(end 322.072 292.7604)
+		(width 2.5)
 		(layer "B.Cu")
 		(net 34)
@@
 	)
 	(segment
-		(start 327.3044 325.2418)
-		(end 327.3044 326.146948)
-		(width 2.5)
-		(layer "B.Cu")
-		(net 34)
-	)
-	(segment
 		(start 291.8968 292.7604)
 		(end 291.8968 292.9636)
@@
 		(layer "B.Cu")
 		(net 34)
-	)
-	(segment
-		(start 327.3044 326.146948)
-		(end 327.3044 297.9928)
-		(width 2.5)
-		(layer "B.Cu")
-		(net 34)
